File: LoRa-V3-PCB.kicad_sch (KiCad schematic)
At the start: 84 parts, among them IC1 SeeedStudio Wio-E5-LE-HF, IC10 BR24G1MFVT-5AE2, IC11 BR24G1MFVT-5AE2, IC12 MCP73123T-22SI/MF, IC2 CP2102N-Axx-xQFN24, IC3 USBLC6-2SC6, IC4 BQ25504RGTR, IC8 BR24G1MFVT-5AE2, IC9 BR24G1MFVT-5AE2, Q1 PJC7400_R1_00001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

Commit message: upgrade workflow
Parts:
- C1, C10, C2, C5, C6, C7, C8, C9: mpn (none) -> CGA3E2X7R1E104K080AA
- C11, C12, C13, C14, C15, C16, C17, C18: mpn (none) -> CL21B475KPFNFNE
- C25, C26, C27: mpn (none) -> CL21B106KPQNNWE
- C30, C31, C32, C33, C34, C35, C36, C37: mpn (none) -> CGA3E1X7R1E105K080AC
- CONN1: mpn (none) -> 217179-0001
- CONN2: mpn (none) -> 2460
- CONN3: mpn (none) -> SM04B-SRSS-TB(LF)(DN)(P)
- CONN4: mpn (none) -> B2B-XH-A(LF)(SN)
- CONN5: mpn (none) -> 73391-0080
- CONN6: mpn (none) -> 2-1734839-4
- CONN7: mpn (none) -> BC075-08-A-L-A
- CONN8, F1, F2, F3, H1, H2, H3, H4, JP1, JP2: mpn (none) -> NA
- D1, D2, D3: mpn (none) -> MSS1P3HM3_A/H
- IC1: mpn (none) -> 114993121
- IC10, IC11, IC8, IC9: mpn (none) -> BR24G1MFVT-5AE2
- IC12: mpn (none) -> MCP73123T-22SI/MF
- IC2: mpn (none) -> CP2102N-A02-GQFN24R
- IC3: mpn (none) -> USBLC6-2SC6
- IC4: mpn (none) -> BQ25504RGTR
- L1: mpn (none) -> VLS3010CX-470M-1
- L2: mpn (none) -> VLS3010CX-220M-1
- Q1: mpn (none) -> PJC7400_R1_00001
- Q2, Q3, Q4: mpn (none) -> SI2367DS-T1-GE3
- R1: mpn (none) -> ERJ-3RQJ2R2V
- R10, R5, R6, R7, R8, R9: mpn (none) -> AC0603DR-075K1L
- R11, R21: mpn (none) -> CRCW06035M36FKEA
- R12: mpn (none) -> CR0603-JW-103ELF
- R13: mpn (none) -> AC0603FR-0722K1L
- R14, R20: mpn (none) -> RC0603FR-074M75L
- R15: mpn (none) -> AC0603FR-0747K5L
- R17, R18: mpn (none) -> AC0603JR-07330KL
- R19: mpn (none) -> RC0603FR-078M45L
- R2: mpn (none) -> RC0603FR-071M69L
- R23: mpn (none) -> RC0603FR-7W330RL
- R3: mpn (none) -> SR0603JR-071KL
- SW1: mpn (none) -> 434331045822
- SW2: mpn (none) -> SLLB510100
